File: VCAbottom.kicad_pcb (KiCad board)
At the start: 2 copper layers, 39 x 100 mm, 49 parts, among them J1 PWR, J2 sigA, J3 sigB, J4 PWR2, Q1 2N3906, Q2 2N3906, U1 TL072, U2 LM13700, U3 TL072

Commit message: Add files via upload
Routing:
- net /CVA: track 48.4 -> 50.9 mm
Other:
- board text added: "Stripey- Stripe"
