File: VCAtop.kicad_pcb (KiCad board)
At the start: 2 copper layers, 39 x 100 mm, 26 parts, among them J1 EnvelopeA, J10 Conn_01x03_Male, J11 PWR, J2 CVA, J3 SignalInA, J4 SignalOutA, J5 Conn_01x03_Male, J6 EnvelopeB, J7 CVB, J8 SignalInB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

Commit message: Add files via upload
Parts:
- J6: value EnvelopeB -> CVB
- J7: value CVB -> EnvB
Connections:
- R3 pad 2: Net-(J2-PadR) -> Net-(J1-PadR)
- RV2 pad 3: Net-(J1-PadR) -> Net-(J2-PadR)
Routing:
- net Net-(J1-PadR): track 30.5 -> 21.2 mm
- net Net-(J2-PadR): track 30.3 -> 31.6 mm

Commit message: Add files via upload
Parts:
- removed C1: CP, Capacitor_THT:CP_Radial_Tantal_D5.0mm_P2.50mm
Routing:
- net GND: track 5.82 -> 0.90 mm
